File: KiCad/1.0/volvo_bt_board/volvo_bt_board.kicad_sch (KiCad schematic)
At the start: 14 parts, among them J1 DB9_Male, J11 Conn_01x02_Female, J12 Conn_01x02_Female, J2 Conn_01x06_Female, J3 Conn_01x09_Female, J4 Conn_01x02_Female, J5 Conn_01x02_Female, J6 Conn_01x01_Female, J7 Conn_01x01_Female, J8 Conn_01x01_Female, J9 Conn_01x01_Female, U1 ESP32-DEVKITC-32D

Commit message: Update pcb, generate gerber
Parts:
- A1: value Arduino_Nano_v3.x -> (none)
- B1: value SPARKFUN_LOGIC_LEVEL_CONVERTER -> (none)
- J1: footprint Connector_Dsub:DSUB-9_Male_Horizontal_P2.77x2.54mm_EdgePinOffset9.40mm -> (none)
- J11, J12, J4, J5: value Conn_01x02_Female -> (none)
- J2: value Conn_01x06_Female -> (none)
- J3: value Conn_01x09_Female -> (none)
- J6, J7, J8, J9: value Conn_01x01_Female -> (none)
Changed lines of the file:
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@@
   )
   (symbol (lib_id "Connector:Conn_01x09_Female") (at 35.56 120.65 180) (unit 1)
-    (in_bom yes) (on_board yes) (fields_autoplaced)
-    (property "Reference" "J3" (id 0) (at 34.29 121.9201 0)
-      (effects (font (size 1.27 1.27)) (justify left))
-    )
-    (property "Value" "Conn_01x09_Female" (id 1) (at 34.29 119.3801 0)
-      (effects (font (size 1.27 1.27)) (justify left))
-    )
+    (in_bom yes) (on_board yes)
+    (property "Reference" "J3" (id 0) (at 36.195 105.41 0))
+    (property "Value" "" (id 1) (at 30.48 120.65 0))
     (property "Footprint" "Connector_PinSocket_2.54mm:PinSocket_1x09_P2.54mm_Vertical" (id 2) (at 35.56 120.65 0)
       (effects (font (size 1.27 1.27)) hide)
@@
       (effects (font (size 1.27 1.27)) (justify right))
     )
-    (property "Value" "Conn_01x01_Female" (id 1) (at 121.92 33.02 0)
+    (property "Value" "" (id 1) (at 121.92 49.53 0)
       (effects (font (size 1.27 1.27)) (justify right))
     )
@@
       (effects (font (size 1.27 1.27)) (justify left))
     )
-    (property "Value" "Conn_01x02_Female" (id 1) (at 135.89 116.2049 90)
+    (property "Value" "" (id 1) (at 135.89 116.2049 90)
       (effects (font (size 1.27 1.27)) (justify left))
     )
@@
   )
   (symbol (lib_id "Connector:Conn_01x06_Female") (at 35.56 144.78 180) (unit 1)
-    (in_bom yes) (on_board yes) (fields_autoplaced)
-    (property "Reference" "J2" (id 0) (at 34.29 144.7801 0)
-      (effects (font (size 1.27 1.27)) (justify left))
-    )
-    (property "Value" "Conn_01x06_Female" (id 1) (at 34.29 142.2401 0)
-      (effects (font (size 1.27 1.27)) (justify left))
-    )
+    (in_bom yes) (on_board yes)
+    (property "Reference" "J2" (id 0) (at 36.195 132.08 0))
+    (property "Value" "" (id 1) (at 45.72 144.78 0))
     (property "Footprint" "Connector_PinSocket_2.54mm:PinSocket_1x06_P2.54mm_Vertical" (id 2) (at 35.56 144.78 0)
       (effects (font (size 1.27 1.27)) hide)
@@
       (effects (font (size 1.27 1.27)) (justify left))
     )
-    (property "Value" "Arduino_Nano_v3.x" (id 1) (at 258.5594 151.13 0)
+    (property "Value" "" (id 1) (at 258.5594 151.13 0)
       (effects (font (size 1.27 1.27)) (justify left))
     )
@@
       (effects (font (size 1.27 1.27)) (justify left))
     )
-    (property "Value" "Conn_01x02_Female" (id 1) (at 54.61 134.62 90)
+    (property "Value" "" (id 1) (at 54.61 134.62 90)
       (effects (font (size 1.27 1.27)) (justify left))
     )
@@
       (effects (font (size 1.143 1.143)))
     )
-    (property "Value" "SPARKFUN_LOGIC_LEVEL_CONVERTER" (id 1) (at 177.8 100.33 0)
+    (property "Value" "" (id 1) (at 177.8 100.33 0)
       (effects (font (size 1.143 1.143)))
     )
@@
       (effects (font (size 1.27 1.27)) (justify right))
     )
-    (property "Value" "Conn_01x01_Female" (id 1) (at 116.84 33.02 0)
+    (property "Value" "" (id 1) (at 116.84 48.26 0)
       (effects (font (size 1.27 1.27)) (justify right))
     )
@@
       (effects (font (size 1.27 1.27)) (justify left))
     )
-    (property "Footprint" "Connector_Dsub:DSUB-9_Male_Horizontal_P2.77x2.54mm_EdgePinOffset9.40mm" (id 2) (at 193.04 45.72 0)
+    (property "Footprint" "" (id 2) (at 193.04 45.72 0)
       (effects (font (size 1.27 1.27)) hide)
     )
@@
       (effects (font (size 1.27 1.27)) (justify left))
     )
-    (property "Value" "Conn_01x02_Female" (id 1) (at 50.8 153.0349 90)
+    (property "Value" "" (id 1) (at 50.8 153.0349 90)
       (effects (font (size 1.27 1.27)) (justify left))
     )
@@
       (effects (font (size 1.27 1.27)) (justify right))
     )
-    (property "Value" "Conn_01x01_Female" (id 1) (at 111.76 33.02 0)
+    (property "Value" "" (id 1) (at 111.76 48.26 0)
       (effects (font (size 1.27 1.27)) (justify right))
     )
@@
   (symbol (lib_id "Connector:Conn_01x02_Female") (at 139.7 120.65 90) (unit 1)
     (in_bom yes) (on_board yes)
-    (property "Reference" "J12" (id 0) (at 138.43 122.5551 90)
-      (effects (font (size 1.27 1.27)) (justify left))
-    )
-    (property "Value" "Conn_01x02_Female" (id 1) (at 148.59 119.38 90)
+    (property "Reference" "J12" (id 0) (at 146.05 123.19 90)
+      (effects (font (size 1.27 1.27)) (justify left))
+    )
+    (property "Value" "" (id 1) (at 143.51 119.38 90)
       (effects (font (size 1.27 1.27)) (justify left))
     )
@@
       (effects (font (size 1.27 1.27)) (justify right))
     )
-    (property "Value" "Conn_01x01_Female" (id 1) (at 106.68 33.02 0)
+    (property "Value" "" (id 1) (at 106.68 48.26 0)
       (effects (font (size 1.27 1.27)) (justify right))
     )
@@
   (symbol_instances
     (path "/6829d496-0d45-4ae6-9026-a7109fe4cccd"
-      (reference "A1") (unit 1) (value "Arduino_Nano_v3.x") (footprint "Module:Arduino_Nano")
+      (reference "A1") (unit 1) (value "Arduino_Nano") (footprint "Module:Arduino_Nano")
     )
     (path "/91540827-f29a-4db9-93cd-f23dfe2b26ce"
-      (reference "B1") (unit 1) (value "SPARKFUN_LOGIC_LEVEL_CONVERTER") (footprint "Boards:SPARKFUN_LOGIC_LEVEL_CONVERTER")
+      (reference "B1") (unit 1) (value "LOGIC_LEVEL_CONVERTER") (footprint "Boards:SPARKFUN_LOGIC_LEVEL_CONVERTER")
     )
     (path "/a64e5559-eb3d-40e1-954d-9d97d65190b8"
-      (reference "J1") (unit 1) (value "DB9_Male") (footprint "Connector_Dsub:DSUB-9_Male_Horizontal_P2.77x2.54mm_EdgePinOffset9.40mm")
+      (reference "J1") (unit 1) (value "DB9_Male") (footprint "Connector_Dsub:DSUB-9_Male_Horizontal_P2.77x2.84mm_EdgePinOffset7.70mm_Housed_MountingHolesOffset9.12mm")
     )
     (path "/67a50d63-11c5-46b7-99b5-df387b113e3a"
-      (reference "J2") (unit 1) (value "Conn_01x06_Female") (footprint "Connector_PinSocket_2.54mm:PinSocket_1x06_P2.54mm_Vertical")
+      (reference "J2") (unit 1) (value "DAC_B") (footprint "Connector_PinSocket_2.54mm:PinSocket_1x06_P2.54mm_Vertical")
     )
     (path "/22bce858-8dc5-49e4-ad0b-2b620fa01bd6"
-      (reference "J3") (unit 1) (value "Conn_01x09_Female") (footprint "Connector_PinSocket_2.54mm:PinSocket_1x09_P2.54mm_Vertical")
+      (reference "J3") (unit 1) (value "DAC_A") (footprint "Connector_PinSocket_2.54mm:PinSocket_1x09_P2.54mm_Vertical")
     )
     (path "/82f305dc-0c88-403f-9558-9b4b96c42dea"
-      (reference "J4") (unit 1) (value "Conn_01x02_Female") (footprint "Connectors:1X02_NO_SILK")
+      (reference "J4") (unit 1) (value "SF0") (footprint "Connectors:1X02_NO_SILK")
     )
     (path "/cf515e29-bd63-488f-a95f-6649591e2e7d"
-      (reference "J5") (unit 1) (value "Conn_01x02_Female") (footprint "Connectors:1X02_NO_SILK")
+      (reference "J5") (unit 1) (value "SF1") (footprint "Connectors:1X02_NO_SILK")
     )
     (path "/d8e33231-9b08-44b7-a93d-65c3383ad690"
-      (reference "J6") (unit 1) (value "Conn_01x01_Female") (footprint "Connector_PinSocket_2.54mm:PinSocket_1x01_P2.54mm_Vertical")
+      (reference "J6") (unit 1) (value "12V") (footprint "Connector_PinSocket_2.54mm:PinSocket_1x01_P2.54mm_Vertical")
     )
     (path "/d4fbcac6-2a03-4de9-a623-f8aed4c629d0"
-      (reference "J7") (unit 1) (value "Conn_01x01_Female") (footprint "Connector_PinSocket_2.54mm:PinSocket_1x01_P2.54mm_Vertical")
+      (reference "J7") (unit 1) (value "GND") (footprint "Connector_PinSocket_2.54mm:PinSocket_1x01_P2.54mm_Vertical")
     )
     (path "/9bebcfbc-cad6-49e6-bf7d-bd003717caf9"
-      (reference "J8") (unit 1) (value "Conn_01x01_Female") (footprint "Connector_PinSocket_2.54mm:PinSocket_1x01_P2.54mm_Vertical")
+      (reference "J8") (unit 1) (value "GND") (footprint "Connector_PinSocket_2.54mm:PinSocket_1x01_P2.54mm_Vertical")
     )
     (path "/2a7b551c-257d-4eff-a30d-59115565c2c6"
-      (reference "J9") (unit 1) (value "Conn_01x01_Female") (footprint "Connector_PinSocket_2.54mm:PinSocket_1x01_P2.54mm_Vertical")
+      (reference "J9") (unit 1) (value "5V") (footprint "Connector_PinSocket_2.54mm:PinSocket_1x01_P2.54mm_Vertical")
     )
     (path "/3681651e-65e4-42da-bbb5-fcd909f52e1d"
-      (reference "J11") (unit 1) (value "Conn_01x02_Female") (footprint "Connectors:1X02_NO_SILK")
+      (reference "J11") (unit 1) (value "A_TX") (footprint "Connectors:1X02_NO_SILK")
     )
     (path "/d8bdf62a-c236-4a8f-8e6c-757145eb487c"
-      (reference "J12") (unit 1) (value "Conn_01x02_Female") (footprint "Connectors:1X02_NO_SILK")
+      (reference "J12") (unit 1) (value "A_RST") (footprint "Connectors:1X02_NO_SILK")
     )
     (path "/9cfe40b8-c15f-4c06-a518-10601ccc0049"
