File: KiCad/1.0/volvo_bt_board/volvo_bt_board.kicad_pcb (KiCad board)
At the start: 2 copper layers, 14 parts, among them J1 DB9_Male, J11 Conn_01x02_Female, J12 Conn_01x02_Female, J2 Conn_01x06_Female, J3 Conn_01x09_Female, J4 Conn_01x02_Female, J5 Conn_01x02_Female, J6 Conn_01x01_Female, J7 Conn_01x01_Female, J8 Conn_01x01_Female, J9 Conn_01x01_Female, U1 ESP32-DEVKITC-32D

Commit message: Update pcb, generate gerber
Parts:
- A1: value Arduino_Nano_v3.x -> Arduino_Nano
- B1: value SPARKFUN_LOGIC_LEVEL_CONVERTER -> LOGIC_LEVEL_CONVERTER
- J1: footprint Connector_Dsub:DSUB-9_Male_Horizontal_P2.77x2.54mm_EdgePinOffset9.40mm -> Connector_Dsub:DSUB-9_Male_Horizontal_P2.77x2.84mm_EdgePinOffset7.70mm_Housed_MountingHolesOffset9.12mm
- J11: value Conn_01x02_Female -> A_TX
- J12: value Conn_01x02_Female -> A_RST
- J2: value Conn_01x06_Female -> DAC_B
- J3: value Conn_01x09_Female -> DAC_A
- J4: value Conn_01x02_Female -> SF0
- J5: value Conn_01x02_Female -> SF1
- J6: value Conn_01x01_Female -> 12V
- J7, J8: value Conn_01x01_Female -> GND
- J9: value Conn_01x01_Female -> 5V
- moved J4 27.1 mm to (93.3, 130.8), turned to -90 degrees
- moved J5 23.1 mm to (87.6, 133.3), turned to 90 degrees
- moved J12 1.27 mm to (146.1, 114.9)
Routing:
- net Net-(J2-Pad4): track 5.08 -> 27.4 mm
- net GND: track 308.7 -> 326.1 mm
- net Net-(J2-Pad2): track 5.08 -> 19.2 mm
- net Net-(J3-Pad2): track 39.8 -> 27.6 mm
- net MELBUS_BUSY: track 193.4 -> 196.8 mm
- net Net-(B1-PadLV4): track 19.6 -> 21.2 mm
- net Net-(J12-Pad1): track 5.11 -> 6.38 mm
- net MELBUS_DATA: track 174.3 -> 173.3 mm
- net AUDIO_R: track 45.9 -> 45.3 mm
- net Net-(B1-PadLV3): track 12.5 -> 13.1 mm

Commit message: Update project
Other:
- board outline added: 134.6 x 99.7 mm
Changed lines of the file:
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@@
     )
   )
+  (gr_rect (start 71.755 41.275) (end 206.375 140.97) (layer "Edge.Cuts") (width 0.1) (fill none))
   (segment locked (start 162.56 83.82) (end 180.34 83.82) (width 1) (layer "F.Cu") (net 48))
   (segment locked (start 180.34 83.82) (end 195.58 83.82) (width 1) (layer "F.Cu") (net 48))
